File: swd-debug-adapter.kicad_pcb (KiCad board)
At the start: 2 copper layers, 63.5 x 38.1 mm, 34 parts, among them J1 JLink, J2 UART, J3 TC2030, J4 WCHLink, J5 FPC, J6 TC2050, J7 DF52, J8 PWR_SEL, J9 PWR_PIN, SW1 RESET, SW2 HIGH, SW3 LOW, U1 XC6206P332MR-G

Commit message: Part export
Parts:
- added kibuzzard-695ABEB9: G***, kibuzzard-695ABEB9, F.Cu at (149.5, 95.2)
- added kibuzzard-695ABEC3: G***, kibuzzard-695ABEC3, F.Cu at (158.5, 90.8)
- added kibuzzard-695ABECD: G***, kibuzzard-695ABECD, F.Cu at (158.5, 99.5)
- added kibuzzard-695ABEEB: G***, kibuzzard-695ABEEB, F.Cu at (168.2, 89.8)
- added kibuzzard-695ABEF1: G***, kibuzzard-695ABEF1, F.Cu at (171.9, 100.8)
- moved J5 11.7 mm to (172.6, 89.8)
- moved J7 10.3 mm to (175.4, 100.8)
- moved R4 9.95 mm to (166.2, 95.2), turned to -90 degrees
- moved R3 9.95 mm to (158.8, 95.2), turned to -90 degrees
- moved kibuzzard-695ABBBA 0.20 mm to (148.6, 107.8)
- moved kibuzzard-695ABBC6 0.20 mm to (162.6, 107.8)
- turned SW2 to 90 degrees
- turned SW3 to 90 degrees
Connections:
- net Net-(D2-K) renamed /5V_REG
Routing:
- net +3V3: track 0.00 -> 119.5 mm
- net /~{RESET}: track 0.00 -> 105.8 mm, vias 0 -> 3
- net /HOST_TX: track 0.00 -> 79.6 mm, vias 0 -> 1
- net /SWCLK: track 16.6 -> 92.3 mm, vias 0 -> 1
- net /SWDIO: track 16.6 -> 89.0 mm, vias 0 -> 1
- net /SWO: track 0.00 -> 58.4 mm, vias 0 -> 1
- net /HOST_RX: track 13.0 -> 63.4 mm
- net +5V: track 0.00 -> 34.2 mm
- net /SW_NLOW: track 0.00 -> 26.6 mm, vias 0 -> 1
- net +3V3_GEN: track 3.89 -> 30.1 mm
- net /SW_NHIGH: track 0.00 -> 17.9 mm, vias 0 -> 1
- net Net-(D1-A): track 0.00 -> 6.12 mm
- net /5V_REG: track 0.00 -> 3.55 mm
- net GND: vias 0 -> 49
- added copper zone on F.Cu, net /5V_REG
- added copper zone on B.Cu, net GND
- added copper zone on F.Cu, net GND
