File: swd-debug-adapter.kicad_sch (KiCad schematic)
At the start: 28 parts, among them J1 JLink, J2 UART, J3 TC2030, J4 WCHLink, J5 FPC, J6 TC2050, J7 DF52, J8 PWR_SEL, J9 PWR_PIN, SW1 RESET, SW2 HIGH, SW3 LOW, U1 XC6206P332MR-G

Commit message: Part export
Parts:
- D1, D5: LCSC Part (none) -> C2286
- R1, R2: LCSC Part (none) -> C25091
- R3, R4: LCSC Part (none) -> C25744
Connections:
- net 5V_REG: now reaches C1.1, C2.1, D2.1 (K), D4.1 (K), U1.3 (VI)
Changed lines of the file:
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@@
 		)
 	)
+	(label "5V_REG"
+		(at 124.46 101.6 180)
+		(effects
+			(font
+				(size 0.635 0.635)
+				(color 132 132 132 1)
+			)
+			(justify right bottom)
+		)
+	)
 	(label "~{RESET}"
 		(at 228.6 104.14 0)
@@
 			)
 		)
+		(property "LCSC Part" "C2286"
+			(at 173.99 104.14 90)
+			(effects
+				(font
+					(size 1.27 1.27)
+				)
+				(hide yes)
+			)
+		)
 		(pin "2"
 		)
@@
 			)
 		)
+		(property "LCSC Part" "C25744"
+			(at 63.5 152.4 0)
+			(effects
+				(font
+					(size 1.27 1.27)
+				)
+				(hide yes)
+			)
+		)
 		(pin "2"
 		)
@@
 			)
 		)
+		(property "LCSC Part" "C25091"
+			(at 190.5 114.3 0)
+			(effects
+				(font
+					(size 1.27 1.27)
+				)
+				(hide yes)
+			)
+		)
 		(pin "2"
 		)
@@
 			)
 		)
+		(property "LCSC Part" "C2286"
+			(at 190.5 104.14 90)
+			(effects
+				(font
+					(size 1.27 1.27)
+				)
+				(hide yes)
+			)
+		)
 		(pin "2"
 		)
@@
 			)
 		)
+		(property "LCSC Part" "C25091"
+			(at 173.99 114.3 0)
+			(effects
+				(font
+					(size 1.27 1.27)
+				)
+				(hide yes)
+			)
+		)
 		(pin "2"
 		)
@@
 			(at 88.9 139.7 0)
 			(effects
+				(font
+					(size 1.27 1.27)
+				)
+				(hide yes)
+			)
+		)
+		(property "LCSC Part" "C25744"
+			(at 88.9 139.7 0)
+			(effects
